File: Schematic/prc1000.sch (EAGLE design)
At the start: 60 parts, among them IC1 4508N, IC2 4556N, IC3 4011N, IC5 HM 6116, T1 2N3904, T2 2N3904, T3 2N3904

Commit message: Updated, ready for review
Parts:
- removed JP1: (no value), pinhead:PINHD-1X12
- added C6: (no value), resistor:C-US050-030X075
- added R16, R17, R18: 8.2K, resistor:R-US_0207/10
Connections:
- net IORQ renamed IOREQ
- removed net IO3?: JP1.6
- removed net LCD0: JP1.2
- removed net LCD1: JP1.3
- removed net LCD2: JP1.4
- removed net LCD3: JP1.5
- removed net N$26: JP6.1
- removed net N$27: JP6.2
- removed net N$28: JP6.3
- removed net N$29: JP6.4
- removed net N$30: JP6.5
- removed net N$31: JP6.6
- removed net N$32: JP6.7
- removed net OE: IC5G$1.!OE, JP1.9
- removed net RD: IC4.RD, JP4.15
- removed net WE: IC4.WR, IC5G$1.!WE, JP1.8
- new net N$11: R17.2, R18.1
- new net RD_Z80: IC4.RD, IC5G$1.!OE, JP4.15, JP6.4
- new net WE_Z80: IC4.WR, IC5G$1.!WE, JP6.5
- net +5V: now also DIS1.VDD, R16.1, R18.2
- net A8: now also DIS1.R/W, JP6.6; no longer JP1.7
- net CLK: now also C5.2, JP6.2; no longer JP1.11
- net D0: now also DIS1.D4
- net D1: now also DIS1.D5
- net D2: now also DIS1.D6
- net D3: now also DIS1.D7, JP6.7
- net GND: now also C5.1, C6.2, DIS1.VSS, JP6.3
- net LCD_UNKNOWN: now also JP6.1; no longer JP1.12
- net N$22: now also C6.1, R16.2
- net N$23: now also R17.1
Other:
- note added: "LCD_R/W"
- moved on the sheet: C3, C5, D4, D5, DIS1, JP4, JP5, JP6, R11, R12, R13, R14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

Commit message: Latest updates 99% done?
Parts:
- removed R10, R3, R4, R6: 8.2K, resistor:R-US_0207/10
Connections:
- net 74157_4I0 renamed LOWROM_CS
- net C1_17 renamed CART_MREQ
- net C2_17 renamed CART_IORQ
- net D0_L08 renamed LOWROM_BANK
- net D1_L08 renamed BANK1
- net D3_L08 renamed CARTSEL
- removed net A16: JP5.7
- removed net C1_18: JP4.18
- new net BANK2: V11.3B
- net +5V: now also IC1P.VDD, IC2P.VDD, IC3P.VDD, V1/+UB.+UB, V2/+UB.+UB, V3/+UB.+UB
- net A13: now also JP5.3; no longer JP5.4
- net A14: no longer JP5.2
- net A14_BIOS: now also JP5.2
- net A15: no longer JP5.3
- net A16_BIOS: now also JP5.7
- net A8: now also JP5.4
- net D2_L08: no longer V11.3B
- net GND: now also IC1P.VSS, IC2P.VSS, IC3P.VSS, V2/-UB.-UB, V3/-UB.-UB
- net RAM_CS: now also JP4.18
Other:
- note added: "ADDR_Latch"
- note added: "CART_IO"
- note added: "KB_latch"
- note added: "LOWROM"
- note added: "MAP_CART"
- note added: "MEM_Latch"
- note removed: "BIOS"
- moved on the sheet: IC2P, IC3P, V1/-UB, V2/+UB, V2/-UB, V3/+UB, V3/-UB
